File: EEOP_Testbed/EEOP_Testbed.kicad_pcb (KiCad board)
At the start: 2 copper layers, 55 x 55 mm, 36 parts, among them J101 Conn_01x09, J201 Conn_01x32, J202 Conn_01x32, Q301 FDS6680A, U101 AS78L05RTR-E1, U201 TXB0104PW, U202 HV507PG-G, U301 LT3750AEMS-TRPBF, U302 DA2032-AL

Commit message: Incorporated design review feedback and updated fab files
Parts:
- Q301: value FDS6680A -> MCQ15N10YA; footprint Touchpoint:SOIC127P600X175-8N -> Package_SO:SOIC-8_3.9x4.9mm_P1.27mm
