File: EEOP_Testbed/Flyback_Converter.kicad_sch (KiCad schematic)
At the start: 18 parts, among them Q301 FDS6680A, U301 LT3750AEMS-TRPBF, U302 DA2032-AL

Commit message: Incorporated design review feedback and updated fab files
Parts:
- Q301: value FDS6680A -> MCQ15N10YA; footprint Touchpoint:SOIC127P600X175-8N -> Package_SO:SOIC-8_3.9x4.9mm_P1.27mm
Changed lines of the file:
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@@
 			)
 		)
-		(property "Value" "FDS6680A"
+		(property "Value" "MCQ15N10YA"
 			(at 116.84 93.9799 0)
 			(effects
@@
 			)
 		)
-		(property "Footprint" "Touchpoint:SOIC127P600X175-8N"
+		(property "Footprint" "Package_SO:SOIC-8_3.9x4.9mm_P1.27mm"
 			(at 111.76 92.71 0)
 			(effects
