File: Hydra_Driver/Driver_Unit.kicad_sch (KiCad schematic)
At the start: 27 parts, among them IC201 DRV8313RHHR, U201 INA4181A3IPWR

Commit message: Incorporated design review feedback and updated fab files
Connections:
- net +3.3V renamed L3V3
