File: Hydra_Driver/Hydra_Driver.kicad_sch (KiCad schematic)
At the start: 41 parts, among them IC101 ESP32-S3-WROOM-1-N4, J101 USB4105-GF-A, J102 Conn_01x02, J103 Conn_01x07, J104 Conn_01x04, J105 Conn_01x03, J107 Conn_01x04, J108 Conn_01x03, J109 Conn_01x02, J110 Conn_01x07, SW101 SW_SPST, SW102 SW_SPST, U101 USBLC6-2SC6, U102 MIC5504-3.3YM5-TR, U103 SN74LVC1G80DBVR

Commit message: Fixed issues preparing for build
Fixed XT30 connectors on Hydra_Driver reversed, fixed I2C connector pin order, refined silkscreens
Connections:
- net +3.3V: now also J104.3 (Pin_3), J107.3 (Pin_3); no longer J104.1 (Pin_1), J107.1 (Pin_1)
- net GND: now also J102.1 (Pin_1), J104.4 (Pin_4), J107.4 (Pin_4), J109.1 (Pin_1); no longer J102.2 (Pin_2), J104.2 (Pin_2), J107.2 (Pin_2), J109.2 (Pin_2)
- net SCL1: now also IC101.30 (IO37), J107.1 (Pin_1); no longer IC101.31 (IO38), J107.4 (Pin_4)
- net SCL2: now also IC101.32 (IO39), J104.1 (Pin_1); no longer IC101.33 (IO40), J104.4 (Pin_4)
- net SDA1: now also IC101.31 (IO38), J107.2 (Pin_2); no longer IC101.30 (IO37), J107.3 (Pin_3)
- net SDA2: now also IC101.33 (IO40), J104.2 (Pin_2); no longer IC101.32 (IO39), J104.3 (Pin_3)
- net VMOT: now also J102.2 (Pin_2), J109.2 (Pin_2); no longer J102.1 (Pin_1), J109.1 (Pin_1)
Other:
- moved on the sheet: J102, J109
