File: Combined_Stencil3/Combined_Stencil3.kicad_pcb (KiCad board)
At the start: 2 copper layers, 149 x 132 mm, 374 parts, among them IC101 AS5600-ASOT, IC101 ESP32-S3-WROOM-1-N4, IC102 AS5600-ASOT, IC103 AS5600-ASOT, IC104 AS5600-ASOT, IC105 AS5600-ASOT, IC106 AS5600-ASOT, IC107 AS5600-ASOT, IC108 AS5600-ASOT, IC109 AS5600-ASOT, IC110 AS5600-ASOT, IC111 AS5600-ASOT, IC112 AS5600-ASOT, IC113 AS5600-ASOT, IC114 AS5600-ASOT, IC115 AS5600-ASOT, IC116 AS5600-ASOT, IC117 AS5600-ASOT, IC118 AS5600-ASOT, IC119 AS5600-ASOT, IC120 AS5600-ASOT, IC121 AS5600-ASOT, IC122 AS5600-ASOT, IC123 AS5600-ASOT, IC124 AS5600-ASOT, IC125 AS5600-ASOT, IC201 DRV8313RHHR, IC301 DRV8313RHHR, J101 Conn_01x04, J101 Conn_01x09, J101 USB4105-GF-A, J102 Conn_01x02, J102 Conn_01x04, J103 Conn_01x04, J103 Conn_01x07, J104 Conn_01x04, J105 Conn_01x03, J105 Conn_01x04, J106 Conn_01x04, J107 Conn_01x04, J108 Conn_01x03, J108 Conn_01x04, J109 Conn_01x02, J109 Conn_01x04, J110 Conn_01x04, J110 Conn_01x07, J111 Conn_01x04, J112 Conn_01x04, J113 Conn_01x04, J114 Conn_01x04, J115 Conn_01x04, J116 Conn_01x04, J117 Conn_01x04, J118 Conn_01x04, J119 Conn_01x04, J120 Conn_01x04, J121 Conn_01x04, J122 Conn_01x04, J123 Conn_01x04, J124 Conn_01x04, J125 Conn_01x04, J201 Conn_01x32, J202 Conn_01x32, Q301 MCQ15N10YA, SW101 SW_SPST, SW102 SW_SPST, U101 AS78L05RTR-E1, U101 USBLC6-2SC6, U102 MIC5504-3.3YM5-TR, U103 SN74LVC1G80DBVR, U201 INA4181A3IPWR, U201 TXB0104PW, U202 HV507PG-G, U301 INA4181A3IPWR, U301 LT3750AEMS-TRPBF, U302 DA2032-AL

Commit message: More changes to start production
Parts:
- removed the R103 at (38.8, 139.5)
- removed the R103 at (87.5, 81.0)
- removed the R106 at (31.5, 25.0)
- removed the R109 at (45.5, 25.0)
- removed R112, R115, R118, R121, R124, R127, R130, R133, R136, R139, R142, R145, R148, R151, R154, R157, R160, R163, R166, R169, R172, R175: 10k, Resistor_SMD:R_0402_1005Metric
- removed the REF** at (25.7, 147.0)
- removed the REF** at (25.7, 123.0)
- removed the REF** at (49.8, 123.0)
- removed the REF** at (49.8, 147.0)
- added R103: 10k, Resistor_SMD:R_0402_1005Metric, F.Cu at (32.8, 138.3)
- added REF**: MountingHole_2.7mm_M2.5, MountingHole:MountingHole_2.7mm_M2.5, F.Cu at (19.8, 145.9)
- added REF**: MountingHole_2.7mm_M2.5, MountingHole:MountingHole_2.7mm_M2.5, F.Cu at (19.8, 121.8)
- added REF**: MountingHole_2.7mm_M2.5, MountingHole:MountingHole_2.7mm_M2.5, F.Cu at (43.8, 121.8)
- added REF**: MountingHole_2.7mm_M2.5, MountingHole:MountingHole_2.7mm_M2.5, F.Cu at (43.8, 145.9)
- moved R102 9.04 mm to (34.3, 129.8), turned to 90 degrees
- moved C101 6.09 mm to (26.0, 131.8)
- moved C102 6.09 mm to (26.8, 133.6)
- moved D101 6.09 mm to (31.8, 121.8)
- moved IC101 6.09 mm to (31.8, 133.8)
- moved J101 6.09 mm to (31.8, 145.8)
- moved R101 6.09 mm to (34.5, 121.8)
- moved R104 6.09 mm to (30.0, 138.3)
- moved JP101 3.24 mm to (37.8, 131.8), turned to 0 degrees
Connections:
- JP101 pad 1: GND -> Net-(IC101-DIR)
- JP101 pad 2: Net-(IC101-DIR) -> +3.3V
- R102 pad 1: +3.3V -> Net-(IC101-DIR)
- R102 pad 2: Net-(IC101-DIR) -> GND
Routing:
- net +3.3V: track 229.2 -> 231.4 mm
Other:
- board size 149 x 132 mm -> 153 x 131.5 mm
- board text added: "CCW"
