File: Hydra_Encoder/Hydra_Encoder.kicad_pcb (KiCad board)
At the start: 2 copper layers, 30 x 30 mm, 14 parts, among them IC101 AS5600-ASOT, J101 Conn_01x04

Commit message: Fixed issues preparing for build
Fixed XT30 connectors on Hydra_Driver reversed, fixed I2C connector pin order, refined silkscreens
Parts:
- moved R104 7.25 mm to (-1.75, 4.50), turned to 0 degrees
- moved R103 2.25 mm to (1.00, 4.50), turned to 180 degrees
- renumbered D2 to D101, R7 to R101, R103 to R102, R101 to R103, R102 to R104
Connections:
- J101 pad 1: +3.3V -> /SCL
- J101 pad 2: GND -> /SDA
- J101 pad 3: /SDA -> +3.3V
- J101 pad 4: /SCL -> GND
Routing:
- net /SCL: track 13.7 -> 12.7 mm
- net GND: track 7.92 -> 7.42 mm

Commit message: More changes to start production
Parts:
- moved JP101 4.78 mm to (6.00, -2.00), turned to 0 degrees
- moved R102 3.20 mm to (2.50, -4.00), turned to 90 degrees
Connections:
- JP101 pad 1: GND -> Net-(IC101-DIR)
- JP101 pad 2: Net-(IC101-DIR) -> +3.3V
- R102 pad 1: +3.3V -> Net-(IC101-DIR)
- R102 pad 2: Net-(IC101-DIR) -> GND
Routing:
- net +3.3V: track 0.00 -> 2.20 mm
Other:
- board text added: "CCW"
