File: Microcoder/Microcoder-panel.kicad_pcb (KiCad board)
At the start: 2 copper layers, 68 x 80 mm, 225 parts, among them IC101 AS5600-ASOT, IC102 AS5600-ASOT, IC103 AS5600-ASOT, IC104 AS5600-ASOT, IC105 AS5600-ASOT, IC106 AS5600-ASOT, IC107 AS5600-ASOT, IC108 AS5600-ASOT, IC109 AS5600-ASOT, IC110 AS5600-ASOT, IC111 AS5600-ASOT, IC112 AS5600-ASOT, IC113 AS5600-ASOT, IC114 AS5600-ASOT, IC115 AS5600-ASOT, IC116 AS5600-ASOT, IC117 AS5600-ASOT, IC118 AS5600-ASOT, IC119 AS5600-ASOT, IC120 AS5600-ASOT, IC121 AS5600-ASOT, IC122 AS5600-ASOT, IC123 AS5600-ASOT, IC124 AS5600-ASOT, IC125 AS5600-ASOT, J101 Conn_01x04, J102 Conn_01x04, J103 Conn_01x04, J104 Conn_01x04, J105 Conn_01x04, J106 Conn_01x04, J107 Conn_01x04, J108 Conn_01x04, J109 Conn_01x04, J110 Conn_01x04, J111 Conn_01x04, J112 Conn_01x04, J113 Conn_01x04, J114 Conn_01x04, J115 Conn_01x04, J116 Conn_01x04, J117 Conn_01x04, J118 Conn_01x04, J119 Conn_01x04, J120 Conn_01x04, J121 Conn_01x04, J122 Conn_01x04, J123 Conn_01x04, J124 Conn_01x04, J125 Conn_01x04

Commit message: Fixed issues preparing for build
Fixed XT30 connectors on Hydra_Driver reversed, fixed I2C connector pin order, refined silkscreens
Connections:
- J101 pad 1: +3.3V -> /SCL
- J101 pad 2: GND -> /SDA
- J101 pad 3: /SDA -> +3.3V
- J101 pad 4: /SCL -> GND
- J102 pad 1: +3.3V -> /SCL
- J102 pad 2: GND -> /SDA
- J102 pad 3: /SDA -> +3.3V
- J102 pad 4: /SCL -> GND
- J103 pad 1: +3.3V -> /SCL
- J103 pad 2: GND -> /SDA
- J103 pad 3: /SDA -> +3.3V
- J103 pad 4: /SCL -> GND
- J104 pad 1: +3.3V -> /SCL
- J104 pad 2: GND -> /SDA
- J104 pad 3: /SDA -> +3.3V
- J104 pad 4: /SCL -> GND
- J105 pad 1: +3.3V -> /SCL
- J105 pad 2: GND -> /SDA
- J105 pad 3: /SDA -> +3.3V
- J105 pad 4: /SCL -> GND
- J106 pad 1: +3.3V -> /SCL
- J106 pad 2: GND -> /SDA
- J106 pad 3: /SDA -> +3.3V
- J106 pad 4: /SCL -> GND
- J107 pad 1: +3.3V -> /SCL
- J107 pad 2: GND -> /SDA
- J107 pad 3: /SDA -> +3.3V
- J107 pad 4: /SCL -> GND
- J108 pad 1: +3.3V -> /SCL
- J108 pad 2: GND -> /SDA
- J108 pad 3: /SDA -> +3.3V
- J108 pad 4: /SCL -> GND
- J109 pad 1: +3.3V -> /SCL
- J109 pad 2: GND -> /SDA
- J109 pad 3: /SDA -> +3.3V
- J109 pad 4: /SCL -> GND
- J110 pad 1: +3.3V -> /SCL
- J110 pad 2: GND -> /SDA
- J110 pad 3: /SDA -> +3.3V
- J110 pad 4: /SCL -> GND
- J111 pad 1: +3.3V -> /SCL
- J111 pad 2: GND -> /SDA
- J111 pad 3: /SDA -> +3.3V
- J111 pad 4: /SCL -> GND
- J112 pad 1: +3.3V -> /SCL
- J112 pad 2: GND -> /SDA
- J112 pad 3: /SDA -> +3.3V
- J112 pad 4: /SCL -> GND
- J113 pad 1: +3.3V -> /SCL
- J113 pad 2: GND -> /SDA
- J113 pad 3: /SDA -> +3.3V
- J113 pad 4: /SCL -> GND
- J114 pad 1: +3.3V -> /SCL
- J114 pad 2: GND -> /SDA
- J114 pad 3: /SDA -> +3.3V
- J114 pad 4: /SCL -> GND
- J115 pad 1: +3.3V -> /SCL
- J115 pad 2: GND -> /SDA
- J115 pad 3: /SDA -> +3.3V
- J115 pad 4: /SCL -> GND
- J116 pad 1: +3.3V -> /SCL
- J116 pad 2: GND -> /SDA
- J116 pad 3: /SDA -> +3.3V
- J116 pad 4: /SCL -> GND
- J117 pad 1: +3.3V -> /SCL
- J117 pad 2: GND -> /SDA
- J117 pad 3: /SDA -> +3.3V
- J117 pad 4: /SCL -> GND
- J118 pad 1: +3.3V -> /SCL
- J118 pad 2: GND -> /SDA
- J118 pad 3: /SDA -> +3.3V
- J118 pad 4: /SCL -> GND
- J119 pad 1: +3.3V -> /SCL
- J119 pad 2: GND -> /SDA
- J119 pad 3: /SDA -> +3.3V
- J119 pad 4: /SCL -> GND
- J120 pad 1: +3.3V -> /SCL
- J120 pad 2: GND -> /SDA
- J120 pad 3: /SDA -> +3.3V
- J120 pad 4: /SCL -> GND
- J121 pad 1: +3.3V -> /SCL
- J121 pad 2: GND -> /SDA
- J121 pad 3: /SDA -> +3.3V
- J121 pad 4: /SCL -> GND
- J122 pad 1: +3.3V -> /SCL
- J122 pad 2: GND -> /SDA
- J122 pad 3: /SDA -> +3.3V
- J122 pad 4: /SCL -> GND
- J123 pad 1: +3.3V -> /SCL
- J123 pad 2: GND -> /SDA
- J123 pad 3: /SDA -> +3.3V
- J123 pad 4: /SCL -> GND
- J124 pad 1: +3.3V -> /SCL
- J124 pad 2: GND -> /SDA
- J124 pad 3: /SDA -> +3.3V
- J124 pad 4: /SCL -> GND
- J125 pad 1: +3.3V -> /SCL
- J125 pad 2: GND -> /SDA
- J125 pad 3: /SDA -> +3.3V
- J125 pad 4: /SCL -> GND
Routing:
- net /SDA: track 235.5 -> 173.2 mm
- net /SCL: track 181.3 -> 210.0 mm
- net GND: track 99.1 -> 96.6 mm

Commit message: More changes to start production
Parts:
- removed R151, R152, R153, R154, R155, R156, R157, R158, R159, R160, R161, R162, R163, R164, R165, R166, R167, R168, R169, R170, R171, R172, R173, R174, R175: 10k, Resistor_SMD:R_0402_1005Metric
- moved R103 77.3 mm to (-23.2, -27.2)
- moved R133 63.9 mm to (-23.2, 14.8)
- moved R121 56.1 mm to (32.8, -13.2)
- moved R143 50.5 mm to (-23.2, 28.8)
- moved R144 50.5 mm to (-23.2, 27.2)
- moved R146 49.7 mm to (-9.25, 27.2)
- moved R113 44.3 mm to (-23.2, -13.2)
- moved R114 44.3 mm to (-23.2, -14.8)
- moved R149 44.3 mm to (18.8, 28.8)
- moved R150 44.3 mm to (18.8, 27.2)
- moved R116 43.8 mm to (-9.25, -14.8)
- moved R122 42.0 mm to (32.8, -14.8)
- moved R119 42.0 mm to (18.8, -13.2)
- moved R120 42.0 mm to (18.8, -14.8)
- moved R145 41.6 mm to (-9.25, 28.8)
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Connections:
- IC101 pad 8: Net-(IC101-DIR) -> GND
- IC102 pad 8: Net-(IC101-DIR) -> GND
- IC103 pad 8: Net-(IC101-DIR) -> GND
- IC104 pad 8: Net-(IC101-DIR) -> GND
- IC105 pad 8: Net-(IC101-DIR) -> GND
- IC106 pad 8: Net-(IC101-DIR) -> GND
- IC107 pad 8: Net-(IC101-DIR) -> GND
- IC108 pad 8: Net-(IC101-DIR) -> GND
- IC109 pad 8: Net-(IC101-DIR) -> GND
- IC110 pad 8: Net-(IC101-DIR) -> GND
- IC111 pad 8: Net-(IC101-DIR) -> GND
- IC112 pad 8: Net-(IC101-DIR) -> GND
- IC113 pad 8: Net-(IC101-DIR) -> GND
- IC114 pad 8: Net-(IC101-DIR) -> GND
- IC115 pad 8: Net-(IC101-DIR) -> GND
- IC116 pad 8: Net-(IC101-DIR) -> GND
- IC117 pad 8: Net-(IC101-DIR) -> GND
- IC118 pad 8: Net-(IC101-DIR) -> GND
- IC119 pad 8: Net-(IC101-DIR) -> GND
- IC120 pad 8: Net-(IC101-DIR) -> GND
- IC121 pad 8: Net-(IC101-DIR) -> GND
- IC122 pad 8: Net-(IC101-DIR) -> GND
- IC123 pad 8: Net-(IC101-DIR) -> GND
- IC124 pad 8: Net-(IC101-DIR) -> GND
- IC125 pad 8: Net-(IC101-DIR) -> GND
- R103 pad 2: Net-(IC101-DIR) -> /SDA
- R104 pad 2: /SDA -> /SCL
- R105 pad 2: /SCL -> /SDA
- R106 pad 2: Net-(IC101-DIR) -> /SCL
- R109 pad 2: Net-(IC101-DIR) -> /SDA
- R110 pad 2: /SDA -> /SCL
- R111 pad 2: /SCL -> /SDA
- R112 pad 2: Net-(IC101-DIR) -> /SCL
- R115 pad 2: Net-(IC101-DIR) -> /SDA
- R116 pad 2: /SDA -> /SCL
- R117 pad 2: /SCL -> /SDA
- R118 pad 2: Net-(IC101-DIR) -> /SCL
- R121 pad 2: Net-(IC101-DIR) -> /SDA
- R122 pad 2: /SDA -> /SCL
- R123 pad 2: /SCL -> /SDA
- R124 pad 2: Net-(IC101-DIR) -> /SCL
- R127 pad 2: Net-(IC101-DIR) -> /SDA
- R128 pad 2: /SDA -> /SCL
- R129 pad 2: /SCL -> /SDA
- R130 pad 2: Net-(IC101-DIR) -> /SCL
- R133 pad 2: Net-(IC101-DIR) -> /SDA
- R134 pad 2: /SDA -> /SCL
- R135 pad 2: /SCL -> /SDA
- R136 pad 2: Net-(IC101-DIR) -> /SCL
- R139 pad 2: Net-(IC101-DIR) -> /SDA
- R140 pad 2: /SDA -> /SCL
- R141 pad 2: /SCL -> /SDA
- R142 pad 2: Net-(IC101-DIR) -> /SCL
- R145 pad 2: Net-(IC101-DIR) -> /SDA
- R146 pad 2: /SDA -> /SCL
- R147 pad 2: /SCL -> /SDA
- R148 pad 2: Net-(IC101-DIR) -> /SCL
Routing:
- net Net-(IC101-DIR): track 45.1 -> 0.00 mm
- net GND: track 96.6 -> 140.7 mm, vias 100 -> 125
